Commit message: fix: ground_truth_odom GroundTruthOdom() call, lowercase base_link, bridge QoS, TF chain complete

File: robot-description/tron2/SF_TRON2A/xacro/robot.urdf.xacro (robot description, xacro)
@@ -17,5 +17,5 @@
   <joint name="base_imu_Joint" type="fixed">
     <origin rpy="0. 0. 0." xyz="0. 0. 0." />
-    <parent link="base_Link" />
+    <parent link="base_link" />
     <child link="base_imu" />
   </joint>
@@ -38,5 +38,5 @@
   </gazebo>
   <!-- Links -->
-  <link name="base_Link">
+  <link name="base_link">
     <inertial>
       <origin xyz="3.85E-03 -0.11E-03 112.54E-03" rpy="0 0 0" />
@@ -346,5 +346,5 @@
   <joint name="proximal_pitch_L_Joint" type="revolute">
     <origin xyz="-0.00044 0.09178 0.05474" rpy="0 0 0" />
-    <parent link="base_Link" />
+    <parent link="base_link" />
     <child link="proximal_pitch_L_Link" />
     <axis xyz="0.0 0.9961947268929313 -0.0871554135479712" />
@@ -381,5 +381,5 @@
   <joint name="proximal_pitch_R_Joint" type="revolute">
     <origin xyz="-0.00044 -0.09178 0.05474" rpy="0 0 0" />
-    <parent link="base_Link" />
+    <parent link="base_link" />
     <child link="proximal_pitch_R_Link" />
     <axis xyz="0.0 0.9961947268929313 0.0871554135479712" />

Commit message: fix: mid360 inverted mount rpy=3.14159; restore vertical min_angle=-7

File: robot-description/tron2/SF_TRON2A/xacro/robot.urdf.xacro (robot description, xacro)
@@ -46,5 +46,5 @@
     </inertial>
     <visual>
-      <origin xyz="0 0 0" rpy="0 0 0" />
+      <origin xyz="0 0 0" rpy="3.14159 0 0" />
       <geometry>
         <mesh filename="package://robot_description/tron2/SF_TRON2A/meshes/base_Link.STL" />
@@ -53,5 +53,5 @@
     </visual>
     <collision>
-      <origin xyz="0 0 0" rpy="0 0 0" />
+      <origin xyz="0 0 0" rpy="3.14159 0 0" />
       <geometry>
         <mesh filename="package://robot_description/tron2/SF_TRON2A/meshes/base_Link.STL" />
@@ -67,5 +67,5 @@
     </inertial>
     <visual>
-      <origin xyz="0 0 0" rpy="0 0 0" />
+      <origin xyz="0 0 0" rpy="3.14159 0 0" />
       <geometry>
         <mesh filename="package://robot_description/tron2/SF_TRON2A/meshes/proximal_pitch_L_Link.STL" />
@@ -74,5 +74,5 @@
     </visual>
     <collision>
-      <origin xyz="0 0 0" rpy="0 0 0" />
+      <origin xyz="0 0 0" rpy="3.14159 0 0" />
       <geometry>
         <mesh filename="package://robot_description/tron2/SF_TRON2A/meshes/proximal_pitch_L_Link.STL" />
@@ -88,5 +88,5 @@
     </inertial>
     <visual>
-      <origin xyz="0 0 0" rpy="0 0 0" />
+      <origin xyz="0 0 0" rpy="3.14159 0 0" />
       <geometry>
         <mesh filename="package://robot_description/tron2/SF_TRON2A/meshes/proximal_roll_L_Link.STL" />
@@ -95,5 +95,5 @@
     </visual>
     <collision>
-      <origin xyz="0 0 0" rpy="0 0 0" />
+      <origin xyz="0 0 0" rpy="3.14159 0 0" />
       <geometry>
         <mesh filename="package://robot_description/tron2/SF_TRON2A/meshes/proximal_roll_L_Link.STL" />
@@ -109,5 +109,5 @@
     </inertial>
     <visual>
-      <origin xyz="0 0 0" rpy="0 0 0" />
+      <origin xyz="0 0 0" rpy="3.14159 0 0" />
       <geometry>
         <mesh filename="package://robot_description/tron2/SF_TRON2A/meshes/proximal_yaw_L_Link.STL" />
@@ -116,5 +116,5 @@
     </visual>
     <collision>
-      <origin xyz="0 0 0" rpy="0 0 0" />
+      <origin xyz="0 0 0" rpy="3.14159 0 0" />
       <geometry>
         <mesh filename="package://robot_description/tron2/SF_TRON2A/meshes/proximal_yaw_L_Link.STL" />
@@ -129,5 +129,5 @@
     </inertial>
     <visual>
-      <origin xyz="0 0 0" rpy="0 0 0" />
+      <origin xyz="0 0 0" rpy="3.14159 0 0" />
       <geometry>
         <mesh filename="package://robot_description/tron2/SF_TRON2A/meshes/knee_L_Link.STL" />
@@ -136,5 +136,5 @@
     </visual>
     <collision>
-      <origin xyz="0 0 0" rpy="0 0 0" />
+      <origin xyz="0 0 0" rpy="3.14159 0 0" />
       <geometry>
         <mesh filename="package://robot_description/tron2/SF_TRON2A/meshes/knee_L_Link.STL" />
@@ -150,5 +150,5 @@
     </inertial>
     <visual>
-      <origin xyz="0 0 0" rpy="0 0 0" />
+      <origin xyz="0 0 0" rpy="3.14159 0 0" />
       <geometry>
         <mesh filename="package://robot_description/tron2/SF_TRON2A/meshes/ankle_pitch_L_Link.STL" />
@@ -157,5 +157,5 @@
     </visual>
     <collision>
-      <origin xyz="0 0 0" rpy="0 0 0" />
+      <origin xyz="0 0 0" rpy="3.14159 0 0" />
       <geometry>
         <mesh filename="package://robot_description/tron2/SF_TRON2A/meshes/ankle_pitch_L_Link.STL" />
@@ -171,5 +171,5 @@
     </inertial>
     <visual>
-      <origin xyz="0 0 0" rpy="0 0 0" />
+      <origin xyz="0 0 0" rpy="3.14159 0 0" />
       <geometry>
         <mesh filename="package://robot_description/tron2/SF_TRON2A/meshes/proximal_pitch_R_Link.STL" />
@@ -178,5 +178,5 @@
     </visual>
     <collision>
-      <origin xyz="0 0 0" rpy="0 0 0" />
+      <origin xyz="0 0 0" rpy="3.14159 0 0" />
       <geometry>
         <mesh filename="package://robot_description/tron2/SF_TRON2A/meshes/proximal_pitch_R_Link.STL" />
@@ -192,5 +192,5 @@
     </inertial>
     <visual>
-      <origin xyz="0 0 0" rpy="0 0 0" />
+      <origin xyz="0 0 0" rpy="3.14159 0 0" />
       <geometry>
         <mesh filename="package://robot_description/tron2/SF_TRON2A/meshes/proximal_roll_R_Link.STL" />
@@ -199,5 +199,5 @@
     </visual>
     <collision>
-      <origin xyz="0 0 0" rpy="0 0 0" />
+      <origin xyz="0 0 0" rpy="3.14159 0 0" />
       <geometry>
         <mesh filename="package://robot_description/tron2/SF_TRON2A/meshes/proximal_roll_R_Link.STL" />
@@ -213,5 +213,5 @@
     </inertial>
     <visual>
-      <origin xyz="0 0 0" rpy="0 0 0" />
+      <origin xyz="0 0 0" rpy="3.14159 0 0" />
       <geometry>
         <mesh filename="package://robot_description/tron2/SF_TRON2A/meshes/proximal_yaw_R_Link.STL" />
@@ -220,5 +220,5 @@
     </visual>
     <collision>
-      <origin xyz="0 0 0" rpy="0 0 0" />
+      <origin xyz="0 0 0" rpy="3.14159 0 0" />
       <geometry>
         <mesh filename="package://robot_description/tron2/SF_TRON2A/meshes/proximal_yaw_R_Link.STL" />
@@ -233,5 +233,5 @@
     </inertial>
     <visual>
-      <origin xyz="0 0 0" rpy="0 0 0" />
+      <origin xyz="0 0 0" rpy="3.14159 0 0" />
       <geometry>
         <mesh filename="package://robot_description/tron2/SF_TRON2A/meshes/knee_R_Link.STL" />
@@ -240,5 +240,5 @@
     </visual>
     <collision>
-      <origin xyz="0 0 0" rpy="0 0 0" />
+      <origin xyz="0 0 0" rpy="3.14159 0 0" />
       <geometry>
         <mesh filename="package://robot_description/tron2/SF_TRON2A/meshes/knee_R_Link.STL" />
@@ -254,5 +254,5 @@
     </inertial>
     <visual>
-      <origin xyz="0 0 0" rpy="0 0 0" />
+      <origin xyz="0 0 0" rpy="3.14159 0 0" />
       <geometry>
         <mesh filename="package://robot_description/tron2/SF_TRON2A/meshes/ankle_pitch_R_Link.STL" />
@@ -261,5 +261,5 @@
     </visual>
     <collision>
-      <origin xyz="0 0 0" rpy="0 0 0" />
+      <origin xyz="0 0 0" rpy="3.14159 0 0" />
       <geometry>
         <mesh filename="package://robot_description/tron2/SF_TRON2A/meshes/ankle_pitch_R_Link.STL" />
@@ -271,5 +271,5 @@
     <parent link="base_imu" />
     <child link="mid360_Link" />
-    <origin xyz="0 0 0" rpy="0 0 0" />
+    <origin xyz="0 0 0" rpy="3.14159 0 0" />
   </joint>
   <link name="mid360_Link">
@@ -337,5 +337,5 @@
             <samples>32</samples>
             <resolution>1</resolution>
-            <min_angle>0.0</min_angle>
+            <min_angle>-0.122173</min_angle>
             <max_angle>0.907571</max_angle>
           </vertical>

Commit message: revert: undo inverted mid360 mount, back to rpy=0 0 0

File: robot-description/tron2/SF_TRON2A/xacro/robot.urdf.xacro (robot description, xacro)
@@ -46,5 +46,5 @@
     </inertial>
     <visual>
-      <origin xyz="0 0 0" rpy="3.14159 0 0" />
+      <origin xyz="0 0 0" rpy="0 0 0" />
       <geometry>
         <mesh filename="package://robot_description/tron2/SF_TRON2A/meshes/base_Link.STL" />
@@ -53,5 +53,5 @@
     </visual>
     <collision>
-      <origin xyz="0 0 0" rpy="3.14159 0 0" />
+      <origin xyz="0 0 0" rpy="0 0 0" />
       <geometry>
         <mesh filename="package://robot_description/tron2/SF_TRON2A/meshes/base_Link.STL" />
@@ -67,5 +67,5 @@
     </inertial>
     <visual>
-      <origin xyz="0 0 0" rpy="3.14159 0 0" />
+      <origin xyz="0 0 0" rpy="0 0 0" />
       <geometry>
         <mesh filename="package://robot_description/tron2/SF_TRON2A/meshes/proximal_pitch_L_Link.STL" />
@@ -74,5 +74,5 @@
     </visual>
     <collision>
-      <origin xyz="0 0 0" rpy="3.14159 0 0" />
+      <origin xyz="0 0 0" rpy="0 0 0" />
       <geometry>
         <mesh filename="package://robot_description/tron2/SF_TRON2A/meshes/proximal_pitch_L_Link.STL" />
@@ -88,5 +88,5 @@
     </inertial>
     <visual>
-      <origin xyz="0 0 0" rpy="3.14159 0 0" />
+      <origin xyz="0 0 0" rpy="0 0 0" />
       <geometry>
         <mesh filename="package://robot_description/tron2/SF_TRON2A/meshes/proximal_roll_L_Link.STL" />
@@ -95,5 +95,5 @@
     </visual>
     <collision>
-      <origin xyz="0 0 0" rpy="3.14159 0 0" />
+      <origin xyz="0 0 0" rpy="0 0 0" />
       <geometry>
         <mesh filename="package://robot_description/tron2/SF_TRON2A/meshes/proximal_roll_L_Link.STL" />
@@ -109,5 +109,5 @@
     </inertial>
     <visual>
-      <origin xyz="0 0 0" rpy="3.14159 0 0" />
+      <origin xyz="0 0 0" rpy="0 0 0" />
       <geometry>
         <mesh filename="package://robot_description/tron2/SF_TRON2A/meshes/proximal_yaw_L_Link.STL" />
@@ -116,5 +116,5 @@
     </visual>
     <collision>
-      <origin xyz="0 0 0" rpy="3.14159 0 0" />
+      <origin xyz="0 0 0" rpy="0 0 0" />
       <geometry>
         <mesh filename="package://robot_description/tron2/SF_TRON2A/meshes/proximal_yaw_L_Link.STL" />
@@ -129,5 +129,5 @@
     </inertial>
     <visual>
-      <origin xyz="0 0 0" rpy="3.14159 0 0" />
+      <origin xyz="0 0 0" rpy="0 0 0" />
       <geometry>
         <mesh filename="package://robot_description/tron2/SF_TRON2A/meshes/knee_L_Link.STL" />
@@ -136,5 +136,5 @@
     </visual>
     <collision>
-      <origin xyz="0 0 0" rpy="3.14159 0 0" />
+      <origin xyz="0 0 0" rpy="0 0 0" />
       <geometry>
         <mesh filename="package://robot_description/tron2/SF_TRON2A/meshes/knee_L_Link.STL" />
@@ -150,5 +150,5 @@
     </inertial>
     <visual>
-      <origin xyz="0 0 0" rpy="3.14159 0 0" />
+      <origin xyz="0 0 0" rpy="0 0 0" />
       <geometry>
         <mesh filename="package://robot_description/tron2/SF_TRON2A/meshes/ankle_pitch_L_Link.STL" />
@@ -157,5 +157,5 @@
     </visual>
     <collision>
-      <origin xyz="0 0 0" rpy="3.14159 0 0" />
+      <origin xyz="0 0 0" rpy="0 0 0" />
       <geometry>
         <mesh filename="package://robot_description/tron2/SF_TRON2A/meshes/ankle_pitch_L_Link.STL" />
@@ -171,5 +171,5 @@
     </inertial>
     <visual>
-      <origin xyz="0 0 0" rpy="3.14159 0 0" />
+      <origin xyz="0 0 0" rpy="0 0 0" />
       <geometry>
         <mesh filename="package://robot_description/tron2/SF_TRON2A/meshes/proximal_pitch_R_Link.STL" />
@@ -178,5 +178,5 @@
     </visual>
     <collision>
-      <origin xyz="0 0 0" rpy="3.14159 0 0" />
+      <origin xyz="0 0 0" rpy="0 0 0" />
       <geometry>
         <mesh filename="package://robot_description/tron2/SF_TRON2A/meshes/proximal_pitch_R_Link.STL" />
@@ -192,5 +192,5 @@
     </inertial>
     <visual>
-      <origin xyz="0 0 0" rpy="3.14159 0 0" />
+      <origin xyz="0 0 0" rpy="0 0 0" />
       <geometry>
         <mesh filename="package://robot_description/tron2/SF_TRON2A/meshes/proximal_roll_R_Link.STL" />
@@ -199,5 +199,5 @@
     </visual>
     <collision>
-      <origin xyz="0 0 0" rpy="3.14159 0 0" />
+      <origin xyz="0 0 0" rpy="0 0 0" />
       <geometry>
         <mesh filename="package://robot_description/tron2/SF_TRON2A/meshes/proximal_roll_R_Link.STL" />
@@ -213,5 +213,5 @@
     </inertial>
     <visual>
-      <origin xyz="0 0 0" rpy="3.14159 0 0" />
+      <origin xyz="0 0 0" rpy="0 0 0" />
       <geometry>
         <mesh filename="package://robot_description/tron2/SF_TRON2A/meshes/proximal_yaw_R_Link.STL" />
@@ -220,5 +220,5 @@
     </visual>
     <collision>
-      <origin xyz="0 0 0" rpy="3.14159 0 0" />
+      <origin xyz="0 0 0" rpy="0 0 0" />
       <geometry>
         <mesh filename="package://robot_description/tron2/SF_TRON2A/meshes/proximal_yaw_R_Link.STL" />
@@ -233,5 +233,5 @@
     </inertial>
     <visual>
-      <origin xyz="0 0 0" rpy="3.14159 0 0" />
+      <origin xyz="0 0 0" rpy="0 0 0" />
       <geometry>
         <mesh filename="package://robot_description/tron2/SF_TRON2A/meshes/knee_R_Link.STL" />
@@ -240,5 +240,5 @@
     </visual>
     <collision>
-      <origin xyz="0 0 0" rpy="3.14159 0 0" />
+      <origin xyz="0 0 0" rpy="0 0 0" />
       <geometry>
         <mesh filename="package://robot_description/tron2/SF_TRON2A/meshes/knee_R_Link.STL" />
@@ -254,5 +254,5 @@
     </inertial>
     <visual>
-      <origin xyz="0 0 0" rpy="3.14159 0 0" />
+      <origin xyz="0 0 0" rpy="0 0 0" />
       <geometry>
         <mesh filename="package://robot_description/tron2/SF_TRON2A/meshes/ankle_pitch_R_Link.STL" />
@@ -261,5 +261,5 @@
     </visual>
     <collision>
-      <origin xyz="0 0 0" rpy="3.14159 0 0" />
+      <origin xyz="0 0 0" rpy="0 0 0" />
       <geometry>
         <mesh filename="package://robot_description/tron2/SF_TRON2A/meshes/ankle_pitch_R_Link.STL" />
@@ -271,5 +271,5 @@
     <parent link="base_imu" />
     <child link="mid360_Link" />
-    <origin xyz="0 0 0" rpy="3.14159 0 0" />
+    <origin xyz="0 0 0" rpy="0 0 0" />
   </joint>
   <link name="mid360_Link">

Commit message: fix: gzclient crash (force_system_render=0) + mid360 LiDAR sensor plugin

File: robot-description/tron2/SF_TRON2A/xacro/robot.urdf.xacro (robot description, xacro)
@@ -267,31 +267,89 @@
     </collision>
   </link>
-  <!-- Livox Mid-360 LiDAR -->
+  <!-- D435 Camera Links -->
+  <link name="d435_Link">
+    <visual>
+      <origin rpy="1.5707963267948966 0 1.5707963267948966" xyz="0.0 -0.0 0" />
+      <geometry>
+        <box size="0.01 0.01 0.001" />
+      </geometry>
+      <material name="camera_red">
+        <color rgba="1.0 0.0 0.0 1.0" />
+      </material>
+    </visual>
+  </link>
+  <joint name="d435_joint" type="fixed">
+    <origin rpy="0 1.063778179 0" xyz="0.12213 0.01759 0.00599" />
+    <parent link="base_imu" />
+    <child link="d435_Link" />
+  </joint>
+  <joint name="d435_optical_joint" type="fixed">
+    <origin rpy="-1.5707963267948966 0 -1.5707963267948966" xyz="0 0 0" />
+    <parent link="d435_Link" />
+    <child link="d435_optical_frame" />
+  </joint>
+  <link name="d435_optical_frame" />
+  <!-- ════════════════════════════════════════════ -->
+  <!-- Rack (LiDAR mount)                          -->
+  <!-- ════════════════════════════════════════════ -->
+  <link name="rack_link">
+    <inertial>
+      <origin xyz="0 0 0.111" rpy="0 0 0"/>
+      <mass value="0.5"/>
+      <inertia ixx="0.005" ixy="0" ixz="0" iyy="0.005" iyz="0" izz="0.005"/>
+    </inertial>
+    <visual>
+      <origin xyz="0 0 0" rpy="0 0 0"/>
+      <geometry>
+        <mesh filename="package://robot_description/tron2/SF_TRON2A/meshes/rack.stl"/>
+      </geometry>
+      <material name="rack_grey">
+        <color rgba="0.5 0.5 0.5 1"/>
+      </material>
+    </visual>
+    <collision>
+      <origin xyz="0 0 0" rpy="0 0 0"/>
+      <geometry>
+        <mesh filename="package://robot_description/tron2/SF_TRON2A/meshes/rack.stl"/>
+      </geometry>
+    </collision>
+  </link>
+  <joint name="rack_joint" type="fixed">
+    <parent link="base_imu"/>
+    <child link="rack_link"/>
+    <origin xyz="0 0 0.2615" rpy="0 0 0"/>
+  </joint>
+  <!-- ════════════════════════════════════════════ -->
+  <!-- Mid-360 LiDAR（倒装：joint rpy 翻转）         -->
+  <!-- ════════════════════════════════════════════ -->
+  <link name="mid360_link">
+    <inertial>
+      <mass value="0.265"/>
+      <origin xyz="0 0 -0.03" rpy="0 0 0"/>
+      <inertia ixx="0.0005" ixy="0" ixz="0" iyy="0.0005" iyz="0" izz="0.0005"/>
+    </inertial>
+    <visual>
+      <origin xyz="0 0 0" rpy="0 0 0"/>
+      <geometry>
+        <mesh filename="package://robot_description/tron2/SF_TRON2A/meshes/mid360.stl"/>
+      </geometry>
+      <material name="dark">
+        <color rgba="0.15 0.15 0.15 1"/>
+      </material>
+    </visual>
+    <collision>
+      <origin xyz="0 0 0" rpy="3.14159 0 0"/>
+      <geometry>
+        <mesh filename="package://robot_description/tron2/SF_TRON2A/meshes/mid360.stl"/>
+      </geometry>
+    </collision>
+  </link>
   <joint name="mid360_joint" type="fixed">
-    <parent link="base_imu" />
-    <child link="mid360_Link" />
-    <origin xyz="0 0 0" rpy="0 0 0" />
-  </joint>
-  <link name="mid360_Link">
-    <visual>
-      <origin xyz="-0.0425 0 -0.04" rpy="0 0 -1.570796" />
-      <geometry>
-        <mesh filename="package://robot_description/tron2/SF_TRON2A/meshes/mid360/mid360.stl" />
-      </geometry>
-      <material name="mid360_mat"><color rgba="0.5 0.5 0.5 1" /></material>
-    </visual>
-    <collision>
-      <origin xyz="-0.0425 0 -0.04" rpy="0 0 0" />
-      <geometry>
-        <mesh filename="package://robot_description/tron2/SF_TRON2A/meshes/mid360/mid360.stl" />
-      </geometry>
-    </collision>
-    <inertial>
-      <origin xyz="0 0 -0.00" rpy="0 0 -1.570796" />
-      <mass value="0.265" />
-      <inertia ixx="0.001" ixy="0" ixz="0" iyy="0.001" iyz="0" izz="0.001" />
-    </inertial>
-  </link>
-  <gazebo reference="mid360_Link">
+    <parent link="rack_link"/>
+    <child link="mid360_link"/>
+    <origin xyz="0 0 0.19" rpy="3.14159 0 0"/>
+  </joint>
+  <!-- Mid-360 LiDAR Gazebo Sensor -->
+  <gazebo reference="mid360_link">
     <sensor type="ray" name="mid360_lidar">
       <pose>0 0 0.15 0 0 0</pose>
@@ -315,32 +373,8 @@
       <plugin name="mid360_lidar_plugin" filename="libgazebo_ros_laser.so">
         <topicName>/scan</topicName>
-        <frameName>mid360_Link</frameName>
-        <output_type>sensor_msgs/LaserScan</output_type>
+        <frameName>mid360_link</frameName>
       </plugin>
     </sensor>
   </gazebo>
-  <!-- D435 Camera Links -->
-  <link name="d435_Link">
-    <visual>
-      <origin rpy="1.5707963267948966 0 1.5707963267948966" xyz="0.0 -0.0 0" />
-      <geometry>
-        <box size="0.01 0.01 0.001" />
-      </geometry>
-      <material name="camera_red">
-        <color rgba="1.0 0.0 0.0 1.0" />
-      </material>
-    </visual>
-  </link>
-  <joint name="d435_joint" type="fixed">
-    <origin rpy="0 1.063778179 0" xyz="0.12213 0.01759 0.00599" />
-    <parent link="base_imu" />
-    <child link="d435_Link" />
-  </joint>
-  <joint name="d435_optical_joint" type="fixed">
-    <origin rpy="-1.5707963267948966 0 -1.5707963267948966" xyz="0 0 0" />
-    <parent link="d435_Link" />
-    <child link="d435_optical_frame" />
-  </joint>
-  <link name="d435_optical_frame" />
   <!-- Joints -->
   <joint name="proximal_pitch_L_Joint" type="revolute">
